Commit message: updates to support loading the robot in gazebo harmonic

File: p2os_urdf/defs/pioneer3at_body.xacro (robot description, xacro)
@@ -27,4 +27,5 @@
 				<geometry>
 					<mesh filename="package://p2os_urdf/meshes/p3at_meshes/chassis.stl"/>
+					<!--<box size="0.4 0.28 0.17"/>-->
 				</geometry>
 		</collision>
@@ -54,5 +55,6 @@
 			<origin xyz="0 0 0" rpy="0 0 0"/>
 			<geometry>
-				<box size="0 0 0"/>
+				<mesh filename="package://p2os_urdf/meshes/p3at_meshes/top.stl"/>
+				<!--<box size="0.01 0.01 0.01"/>-->
 			</geometry>
 		</collision>
@@ -83,10 +85,4 @@
 			</material>
 		</visual>
-		<collision>
-			<origin xyz="0 0 0" rpy="0 0 0"/>
-			<geometry>
-				<box size="0 0 0"/>
-			</geometry>
-		</collision>
 	</link>
 	<gazebo reference="front_sonar">
@@ -114,10 +110,4 @@
 			</material>
 		</visual>
-		<collision>
-			<origin xyz="0 0 0" rpy="0 0 0"/>
-			<geometry>
-				<box size="0 0 0"/>
-			</geometry>
-		</collision>
 	</link>
 	<gazebo reference="back_sonar">
@@ -150,5 +140,6 @@
 		<origin xyz="0 0 0" rpy="0 0 0"/>
 		<geometry>
-			<box size="0 0 0"/>
+			<mesh filename="package://p2os_urdf/meshes/p3at_meshes/axle.stl"/>
+			<!--<box size="0.01 0.01 0.01"/>-->
 		</geometry>
 	</collision>
@@ -181,5 +172,5 @@
 		<origin xyz="0 0 0" rpy="0 0 0"/>
 		<geometry>
-			<box size="0 0 0"/>
+			<mesh filename="package://p2os_urdf/meshes/p3at_meshes/${suffix}_hubcap.stl"/>
 		</geometry>
 	</collision>
@@ -252,4 +243,5 @@
 		<geometry>
 			<mesh filename="package://p2os_urdf/meshes/p3at_meshes/axle.stl"/>
+			<!--<box size="0.01 0.01 0.01"/>-->
 		</geometry>
 	</collision>
