Commit message: xacro and launch file improvements
added the ability to prefix the robot_description and tf tree components with a namespace to allow multiple robots to be active at the same time
switched to a wireless gamepad/joystick for local control

File: p2os_urdf/defs/pioneer3at.xacro (robot description, xacro)
@@ -5,9 +5,12 @@
        xmlns:xacro="http://ros.org/wiki/xacro"
 name="pioneer3at">
+<!-- Declare Arguments with Default Values -->
+<xacro:arg name="prefix" default=""/>
 <xacro:include filename="$(find p2os_urdf)/defs/pioneer3at_body.xacro"/>
-<xacro:p3at_front suffix="left" reflect="1"/>
-<xacro:p3at_front suffix="right" reflect="-1"/>
-<xacro:p3at_back suffix="left" reflect="1"/>
-<xacro:p3at_back suffix="right" reflect="-1"/>
-<xacro:p3at_gazebo_ext/>
+<xacro:p3at_chassis prefix="$(arg prefix)"/>
+<xacro:p3at_front prefix="$(arg prefix)" suffix="left" reflect="1"/>
+<xacro:p3at_front prefix="$(arg prefix)" suffix="right" reflect="-1"/>
+<xacro:p3at_back prefix="$(arg prefix)" suffix="left" reflect="1"/>
+<xacro:p3at_back prefix="$(arg prefix)" suffix="right" reflect="-1"/>
+<xacro:p3at_gazebo_ext prefix="$(arg prefix)"/>
 </robot>

File: p2os_urdf/defs/pioneer3at_body.xacro (robot description, xacro)
@@ -5,6 +5,8 @@
        xmlns:xacro="http://ros.org/wiki/xacro"
 >
+<xacro:property name="prefix" value="${prefix:=''}" />
 <!-- Chassis -->
-	<link name="base_link">
+<xacro:macro name="p3at_chassis" params="prefix">
+	<link name="${prefix}base_link">
 		<inertial>
 			<mass value="10.0"/>
@@ -31,9 +33,9 @@
 		</collision>
 	</link>
-	<gazebo reference="base_link">
+	<gazebo reference="${prefix}base_link">
 		<material value="Gazebo/Red"/>
 	</gazebo>
 <!-- Top -->
-	<link name="top_plate">
+	<link name="${prefix}top_plate">
 		<inertial>
 			<mass value="0.1"/>
@@ -60,14 +62,14 @@
 		</collision>
 	</link>
-	<gazebo reference="top_plate">
+	<gazebo reference="${prefix}top_plate">
 		<material value="Gazebo/Black"/>
 	</gazebo>
-	<joint name="base_top_joint" type="fixed">
+	<joint name="${prefix}base_top_joint" type="fixed">
 		<origin xyz="0.003 0 0.274" rpy="0 0 0"/>
-		<parent link="base_link"/>
-		<child link="top_plate"/>
+		<parent link="${prefix}base_link"/>
+		<child link="${prefix}top_plate"/>
 	</joint>
 <!-- Front + Back Sonar -->
-	<link name="front_sonar">
+	<link name="${prefix}front_sonar">
 		<inertial>
 			<mass value="0.1"/>
@@ -86,13 +88,13 @@
 		</visual>
 	</link>
-	<gazebo reference="front_sonar">
+	<gazebo reference="${prefix}front_sonar">
 		<material value="Gazebo/Yellow"/>
 	</gazebo>
-	<joint name="base_front_joint" type="fixed">
+	<joint name="${prefix}base_front_joint" type="fixed">
 		<origin xyz="0.193 0 0.25" rpy="0 0 0"/>
-		<parent link="base_link"/>
-		<child link="front_sonar"/>
-	</joint>
-	<link name="back_sonar">
+		<parent link="${prefix}base_link"/>
+		<child link="${prefix}front_sonar"/>
+	</joint>
+	<link name="${prefix}back_sonar">
 		<inertial>
 			<mass value="0.1"/>
@@ -111,15 +113,16 @@
 		</visual>
 	</link>
-	<gazebo reference="back_sonar">
+	<gazebo reference="${prefix}back_sonar">
 		<material value="Gazebo/Yellow"/>
 	</gazebo>
-	<joint name="base_back_joint" type="fixed">
+	<joint name="${prefix}base_back_joint" type="fixed">
 		<origin xyz="-0.187 0 0.247" rpy="0 0 0"/>
-		<parent link="base_link"/>
-		<child link="back_sonar"/>
-	</joint>
+		<parent link="${prefix}base_link"/>
+		<child link="${prefix}back_sonar"/>
+	</joint>
+</xacro:macro> <!-- End of Chassis -->
 <!-- Front Axles + Wheels + Hubcaps -->
-<xacro:macro name="p3at_front" params="suffix reflect">
-	<link name="p3at_front_${suffix}_axle">
+<xacro:macro name="p3at_front" params="prefix suffix reflect">
+	<link name="${prefix}p3at_front_${suffix}_axle">
 		<inertial>
 			<mass value="0.1"/>
@@ -145,13 +148,13 @@
 	</collision>
 	</link>
-	<gazebo reference="p3at_front_${suffix}_axle">
+	<gazebo reference="${prefix}p3at_front_${suffix}_axle">
 		<material value="Gazebo/Grey"/>
 	</gazebo>
-	<joint name="base_front_${suffix}_axle_joint" type="fixed">
+	<joint name="${prefix}base_front_${suffix}_axle_joint" type="fixed">
 		<origin xyz="0.135 ${reflect*0.156} 0.111" rpy="0 0 0"/>
-		<parent link="base_link"/>
-		<child link="p3at_front_${suffix}_axle"/>
-	</joint>
-	<link name="p3at_front_${suffix}_hub">
+		<parent link="${prefix}base_link"/>
+		<child link="${prefix}p3at_front_${suffix}_axle"/>
+	</joint>
+	<link name="${prefix}p3at_front_${suffix}_hub">
 		<inertial>
 			<mass value="0.1"/>
@@ -176,13 +179,13 @@
 	</collision>
 	</link>
-	<gazebo reference="p3at_front_${suffix}_hub">
+	<gazebo reference="${prefix}p3at_front_${suffix}_hub">
 		<material value="Gazebo/Yellow"/>
 	</gazebo>
-	<joint name="base_front_${suffix}_hub_joint" type="fixed">
+	<joint name="${prefix}base_front_${suffix}_hub_joint" type="fixed">
 		<origin xyz="0 ${reflect*0.041} 0" rpy="0 0 0"/>
-		<parent link="p3at_front_${suffix}_axle"/>
-		<child link="p3at_front_${suffix}_hub"/>
-	</joint>
-	<link name="p3at_front_${suffix}_wheel">
+		<parent link="${prefix}p3at_front_${suffix}_axle"/>
+		<child link="${prefix}p3at_front_${suffix}_hub"/>
+	</joint>
+	<link name="${prefix}p3at_front_${suffix}_wheel">
 		<inertial>
 			<mass value="0.5"/>
@@ -208,8 +211,8 @@
 	</collision>
 	</link>
-	<gazebo reference="p3at_front_${suffix}_wheel">
+	<gazebo reference="${prefix}p3at_front_${suffix}_wheel">
 		<material value="Gazebo/Black"/>
 	</gazebo>
-	<joint name="p3at_front_${suffix}_wheel_joint" type="continuous">
+	<joint name="${prefix}p3at_front_${suffix}_wheel_joint" type="continuous">
   	<axis xyz="0 1 0"/>
     <anchor xyz="0 0 0"/>
@@ -217,11 +220,11 @@
     <joint_properties damping="0.7"/>
 		<origin xyz="0 0 0" rpy="0 0 0"/>
-		<parent link="p3at_front_${suffix}_hub"/>
-		<child link="p3at_front_${suffix}_wheel"/>
+		<parent link="${prefix}p3at_front_${suffix}_hub"/>
+		<child link="${prefix}p3at_front_${suffix}_wheel"/>
 	</joint>
 </xacro:macro>
 <!-- Back Axles + Wheels + Hubcaps -->
-<xacro:macro name="p3at_back" params="suffix reflect">
-	<link name="p3at_back_${suffix}_axle">
+<xacro:macro name="p3at_back" params="prefix suffix reflect">
+	<link name="${prefix}p3at_back_${suffix}_axle">
 		<inertial>
 			<mass value="0.1"/>
@@ -247,13 +250,13 @@
 	</collision>
 	</link>
-	<gazebo reference="p3at_back_${suffix}_axle">
+	<gazebo reference="${prefix}p3at_back_${suffix}_axle">
 		<material value="Gazebo/Grey"/>
 	</gazebo>
-	<joint name="bp3at_back_${suffix}_axle_joint" type="fixed">
+	<joint name="${prefix}bp3at_back_${suffix}_axle_joint" type="fixed">
 		<origin xyz="-0.134 ${reflect*0.156} 0.111" rpy="0 0 0"/>
-		<parent link="base_link"/>
-		<child link="p3at_back_${suffix}_axle"/>
-	</joint>
-	<link name="p3at_back_${suffix}_hub">
+		<parent link="${prefix}base_link"/>
+		<child link="${prefix}p3at_back_${suffix}_axle"/>
+	</joint>
+	<link name="${prefix}p3at_back_${suffix}_hub">
 		<inertial>
 			<mass value="0.1"/>
@@ -276,13 +279,13 @@
 	</collision>
 	</link>
-	<gazebo reference="p3at_back_${suffix}_hub">
+	<gazebo reference="${prefix}p3at_back_${suffix}_hub">
 		<material value="Gazebo/Yellow"/>
 	</gazebo>
-	<joint name="p3at_back_${suffix}_hub_joint" type="fixed">
+	<joint name="${prefix}p3at_back_${suffix}_hub_joint" type="fixed">
 		<origin xyz="-0 ${reflect*0.041} 0" rpy="0 0 0"/>
-		<parent link="p3at_back_${suffix}_axle"/>
-		<child link="p3at_back_${suffix}_hub"/>
-	</joint>
-	<link name="p3at_back_${suffix}_wheel">
+		<parent link="${prefix}p3at_back_${suffix}_axle"/>
+		<child link="${prefix}p3at_back_${suffix}_hub"/>
+	</joint>
+	<link name="${prefix}p3at_back_${suffix}_wheel">
 		<inertial>
 			<mass value="0.5"/>
@@ -306,8 +309,8 @@
 	</collision>
 	</link>
-	<gazebo reference="p3at_back_${suffix}_wheel">
+	<gazebo reference="${prefix}p3at_back_${suffix}_wheel">
 		<material value="Gazebo/Black"/>
 	</gazebo>
-	<joint name="p3at_back_${suffix}_wheel_joint" type="continuous">
+	<joint name="${prefix}p3at_back_${suffix}_wheel_joint" type="continuous">
 	  <axis xyz="0 1 0"/>
     <anchor xyz="0 0 0"/>
@@ -315,8 +318,8 @@
     <joint_properties damping="0.7"/>
 		<origin xyz="0 0 0" rpy="0 0 0"/>
-		<parent link="p3at_back_${suffix}_hub"/>
-		<child link="p3at_back_${suffix}_wheel"/>
-	</joint>
-  <gazebo reference="p3at_back_${suffix}_wheel">
+		<parent link="${prefix}p3at_back_${suffix}_hub"/>
+		<child link="${prefix}p3at_back_${suffix}_wheel"/>
+	</joint>
+  <gazebo reference="${prefix}p3at_back_${suffix}_wheel">
     <kp>1000000.0</kp> <!-- kp and kd for rubber -->
     <kd>100.0</kd>
@@ -327,5 +330,5 @@
     <minDepth>0.00</minDepth>
   </gazebo>
-  <gazebo reference="p3at_front_${suffix}_wheel">
+  <gazebo reference="${prefix}p3at_front_${suffix}_wheel">
     <kp>1000000.0</kp> <!-- kp and kd for rubber -->
     <kd>100.0</kd>
@@ -337,5 +340,5 @@
   </gazebo>
 </xacro:macro>
-<xacro:macro name="p3at_gazebo_ext">
+<xacro:macro name="p3at_gazebo_ext" params="prefix">
 <gazebo>
   <plugin
